Commit message: my_robot/urdf/my_robot.gazebo

File: my_robot/urdf/my_robot.xacro (robot description, xacro)
@@ -4,5 +4,5 @@
   <link name="base_link"></link>
   <joint name="base_link_joint" type="fixed">
-    <origin xyz="0 0 0" rpy="0 0 0"/>
+    <origin xyz="0 0 0.11" rpy="0 0 0"/>
     <parent link="base_link"/>
     <child link="chassis"/>
@@ -76,7 +76,7 @@
       <origin xyz="0 0 0" rpy="0 0 0"/>
       <inertia
-          ixx="0.0031" ixy="0" ixz="0"
-          iyy="0.0031" iyz="0"
-          izz="0.0038"
+          ixx="0.0049" ixy="0" ixz="0"
+          iyy="0.0049" iyz="0"
+          izz="0.0074"
       />
     </inertial>
@@ -107,7 +107,7 @@
       <origin xyz="0 0 0" rpy="0 0 0"/>
       <inertia
-          ixx="0.0031" ixy="0" ixz="0"
-          iyy="0.0031" iyz="0"
-          izz="0.0038"
+          ixx="0.0049" ixy="0" ixz="0"
+          iyy="0.0049" iyz="0"
+          izz="0.0074"
       />
     </inertial>
@@ -138,7 +138,7 @@
       <origin xyz="0 0 0" rpy="0 0 0"/>
       <inertia
-          ixx="0.0031" ixy="0" ixz="0"
-          iyy="0.0031" iyz="0"
-          izz="0.0038"
+          ixx="0.0049" ixy="0" ixz="0"
+          iyy="0.0049" iyz="0"
+          izz="0.0074"
       />
     </inertial>
